Commit message: leader3215 set zero

File: ros/src/arm8_realman_leader/leader_3215_description/urdf/leader_3215_description.xacro (robot description, xacro)
@@ -48,5 +48,5 @@
     <parent link="base_link" />
     <child link="link1" />
-    <axis xyz="0 0 1" />
+    <axis xyz="0 0 -1" />
     <limit lower="-3.14" upper="3.14" effort="0" velocity="0" />
   </joint>
@@ -106,5 +106,5 @@
     <parent link="link2" />
     <child link="link3" />
-    <axis xyz="0 0 1" />
+    <axis xyz="0 0 -1" />
     <limit lower="-3.14" upper="3.14" effort="0" velocity="0" />
   </joint>
@@ -164,5 +164,5 @@
     <parent link="link4" />
     <child link="link5" />
-    <axis xyz="0 0 1" />
+    <axis xyz="0 0 -1" />
     <limit lower="-3.14" upper="3.14" effort="0" velocity="0" />
   </joint>
@@ -222,5 +222,5 @@
     <parent link="link6" />
     <child link="link7" />
-    <axis xyz="0 0 1" />
+    <axis xyz="0 0 -1" />
     <limit lower="-3.14" upper="3.14" effort="0" velocity="0" />
   </joint>
